File: kh-gift-hw.kicad_sch (KiCad schematic)
At the start: 69 parts, among them J2 Conn_01x14, J3 USB, Q1 MMBT5550, Q4 MMBT2222A, Q5 MMBT2222A, SW1 SW_Push, SW2 SW_Push, SW3 SW_Push, U1 DHT11, U10 IRLML0030, U12 IRLML0030, U2 ESP32-WROVER, U3 TP4056, U4 DW01A, U6 CP2102N-Axx-xQFN28, U7 SX1308, U8 AMS1117-3.3, U9 DS1307Z+, Y1 32768 kHz

Commit message: update pcb
Parts:
- Y1: footprint Crystal:Crystal_SMD_3215-2Pin_3.2x1.5mm -> footprints:Crystal_SMD_3215-2Pin_3.2x1.5mm
Connections:
- net LCD_CLK: now also J2.10 (Pin_10)
- net LCD_MISO: now also J2.13 (Pin_13)
- net LCD_MOSI: now also J2.12 (Pin_12)
- net TOUCH_CS: now reaches U2.23 (IO15)
- net TOUCH_CS: now also J2.11 (Pin_11)
- net TOUCH_IRQ: now reaches U2.29 (IO5)
- net TOUCH_IRQ: now also J2.14 (Pin_14)
- no-connect marks 12 -> 7
Other:
- note removed: "OUTLINE"
Changed lines of the file:
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@@
   )
   (no_connect (at 200.025 145.415))
-  (no_connect (at 269.24 100.33))
-  (no_connect (at 269.24 97.79))
   (no_connect (at 75.565 89.535))
   (no_connect (at 75.565 92.075))
-  (no_connect (at 269.24 105.41))
-  (no_connect (at 269.24 102.87))
   (no_connect (at 31.115 86.995))
   (no_connect (at 31.115 84.455))
-  (no_connect (at 269.24 107.95))
   (no_connect (at 75.565 86.995))
   (no_connect (at 31.115 89.535))
@@
     (fill (type none))
   )
-  (rectangle (start 125.73 166.37) (end 174.625 195.58)
-    (stroke (width 1) (type default))
-    (fill (type none))
-  )
   (rectangle (start 114.3 13.97) (end 217.17 113.03)
     (stroke (width 1) (type default))
@@
     (effects (font (size 3.9878 3.9878) (thickness 0.7976) bold) (justify left bottom))
   )
-  (text "OUTLINE" (at 127 194.31 0)
-    (effects (font (size 3.9878 3.9878) (thickness 0.7976) bold) (justify left bottom))
-  )
   (global_label "ESP32_SDA" (shape input) (at 236.22 43.18 180)
     (effects (font (size 1.27 1.27)) (justify right))
@@
     )
   )
+  (global_label "LCD_CLK" (shape input) (at 269.24 97.79 180)
+    (effects (font (size 1.27 1.27)) (justify right))
+    (property "Intersheetrefs" "${INTERSHEET_REFS}" (at 269.24 97.79 0)
+      (effects (font (size 1.27 1.27)) hide)
+    )
+  )
   (global_label "BUTTON" (shape input) (at 31.115 56.515 180)
     (effects (font (size 1.27 1.27)) (justify right))
@@
     )
   )
+  (global_label "LCD_MOSI" (shape input) (at 269.24 102.87 180)
+    (effects (font (size 1.27 1.27)) (justify right))
+    (property "Intersheetrefs" "${INTERSHEET_REFS}" (at 269.24 102.87 0)
+      (effects (font (size 1.27 1.27)) hide)
+    )
+  )
+  (global_label "TOUCH_CS" (shape input) (at 269.24 100.33 180)
+    (effects (font (size 1.27 1.27)) (justify right))
+    (property "Intersheetrefs" "${INTERSHEET_REFS}" (at 269.24 100.33 0)
+      (effects (font (size 1.27 1.27)) hide)
+    )
+  )
   (global_label "CP2102_DTR" (shape input) (at 171.45 53.34 0) (fields_autoplaced)
     (effects (font (size 1.27 1.27)) (justify left))
@@
     )
   )
+  (global_label "TOUCH_IRQ" (shape input) (at 75.565 69.215 0)
+    (effects (font (size 1.27 1.27)) (justify left))
+    (property "Intersheetrefs" "${INTERSHEET_REFS}" (at 75.565 69.215 0)
+      (effects (font (size 1.27 1.27)) hide)
+    )
+  )
   (global_label "LCD_RST" (shape input) (at 269.24 82.55 180)
     (effects (font (size 1.27 1.27)) (justify right))
@@
     )
   )
+  (global_label "TOUCH_CS" (shape input) (at 75.565 84.455 0)
+    (effects (font (size 1.27 1.27)) (justify left))
+    (property "Intersheetrefs" "${INTERSHEET_REFS}" (at 75.565 84.455 0)
+      (effects (font (size 1.27 1.27)) hide)
+    )
+  )
   (global_label "CP2102_DTR" (shape input) (at 192.405 64.77 180) (fields_autoplaced)
     (effects (font (size 1.27 1.27)) (justify right))
@@
     )
   )
+  (global_label "TOUCH_IRQ" (shape input) (at 269.24 107.95 180)
+    (effects (font (size 1.27 1.27)) (justify right))
+    (property "Intersheetrefs" "${INTERSHEET_REFS}" (at 269.24 107.95 0)
+      (effects (font (size 1.27 1.27)) hide)
+    )
+  )
   (global_label "FLASH_EN" (shape input) (at 31.115 48.895 180)
     (effects (font (size 1.27 1.27)) (justify right))
@@
     (effects (font (size 1.27 1.27)) (justify left))
     (property "Intersheetrefs" "${INTERSHEET_REFS}" (at 75.565 64.135 0)
+      (effects (font (size 1.27 1.27)) hide)
+    )
+  )
+  (global_label "LCD_MISO" (shape input) (at 269.24 105.41 180)
+    (effects (font (size 1.27 1.27)) (justify right))
+    (property "Intersheetrefs" "${INTERSHEET_REFS}" (at 269.24 105.41 0)
       (effects (font (size 1.27 1.27)) hide)
     )
@@
       (effects (font (size 1.27 1.27)) (justify left))
     )
-    (property "Footprint" "Crystal:Crystal_SMD_3215-2Pin_3.2x1.5mm" (at 240.03 49.53 0)
-      (effects (font (size 1.27 1.27)) hide)
-    )
+    (property "Footprint" "footprints:Crystal_SMD_3215-2Pin_3.2x1.5mm" (at 240.03 49.53 0)
+      (effects (font (size 1.27 1.27)) hide)
+    )

Commit message: update footprint
Parts:
- BT2: footprint footprints:BAT_CR1220_Holder -> Footprint-Kicad:BAT_CR1220_Holder
- D5, D6, SW3: footprint footprints:JST_EH_S2B-EH_1x02_P2.5mm_Horizontal -> Footprint-Kicad:Connector_ZH_1x02_P1.25mm_Horizontal
- RV1: footprint footprints:JST_EH_S3B-EH_1x03_P2.5mm_Horizontal -> Footprint-Kicad:Connector_ZH_1x03_P1.25mm_Horizontal
- U1: footprint footprints:SNR4-2.54-15.5X12.0X5.5MM -> Footprint-Kicad:SNR4-2.54-15.5X12.0X5.5MM
- U2: footprint footprints:ESP32-WROVER -> Footprint-Kicad:ESP32-WROVER
Changed lines of the file:
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@@
 (kicad_sch
-	(version 20231120)
+	(version 20250114)
 	(generator "eeschema")
-	(generator_version "8.0")
+	(generator_version "9.0")
 	(paper "A4")
+	(rectangle
+		(start 219.71 67.945)
+		(end 282.575 113.03)
+		(stroke
+			(width 1)
+			(type default)
+		)
+		(fill
+			(type none)
+		)
+	)
+	(rectangle
+		(start 14.605 13.97)
+		(end 111.76 113.03)
+		(stroke
+			(width 1)
+			(type default)
+		)
+		(fill
+			(type none)
+		)
+	)
+	(rectangle
+		(start 14.605 166.37)
+		(end 67.31 195.58)
+		(stroke
+			(width 1)
+			(type default)
+		)
+		(fill
+			(type none)
+		)
+	)
+	(rectangle
+		(start 114.3 13.97)
+		(end 217.17 113.03)
+		(stroke
+			(width 1)
+			(type default)
+		)
+		(fill
+			(type none)
+		)
+	)
+	(rectangle
+		(start 14.605 116.205)
+		(end 282.575 163.195)
+		(stroke
+			(width 1)
+			(type default)
+		)
+		(fill
+			(type none)
+		)
+	)
+	(rectangle
+		(start 219.71 13.97)
+		(end 282.575 65.405)
+		(stroke
+			(width 1)
+			(type default)
+		)
+		(fill
+			(type none)
+		)
+	)
+	(rectangle
+		(start 70.485 166.37)
+		(end 123.19 195.58)
+		(stroke
+			(width 1)
+			(type default)
+		)
+		(fill
+			(type none)
+		)
+	)
+	(text "ESP32"
+		(exclude_from_sim no)
+		(at 15.875 111.125 0)
+		(effects
+			(font
+				(size 3.9878 3.9878)
+				(thickness 0.7976)
+				(bold yes)
+			)
+			(justify left bottom)
+		)
+	)
+	(text "RTC"
+		(exclude_from_sim no)
+		(at 220.98 63.5 0)
+		(effects
+			(font
+				(size 3.9878 3.9878)
+				(thickness 0.7976)
+				(bold yes)
+			)
+			(justify left bottom)
+		)
+	)
+	(text "POWER SUPPLY"
+		(exclude_from_sim no)
+		(at 15.875 161.925 0)
+		(effects
+			(font
+				(size 3.9878 3.9878)
+				(thickness 0.7976)
+				(bold yes)
+			)
+			(justify left bottom)
+		)
+	)
+	(text "DHT11"
+		(exclude_from_sim no)
+		(at 15.875 194.31 0)
+		(effects
+			(font
+				(size 3.9878 3.9878)
+				(thickness 0.7976)
+				(bold yes)
+			)
+			(justify left bottom)
+		)
+	)
+	(text "ILI9341"
+		(exclude_from_sim no)
+		(at 221.615 111.125 0)
+		(effects
+			(font
+				(size 3.9878 3.9878)
+				(thickness 0.7976)
+				(bold yes)
+			)
+			(justify left bottom)
+		)
+	)
+	(text "BUZZER"
+		(exclude_from_sim no)
+		(at 71.755 193.675 0)
+		(effects
+			(font
+				(size 3.9878 3.9878)
+				(thickness 0.7976)
+				(bold yes)
+			)
+			(justify left bottom)
+		)
+	)
+	(text "CP2102"
+		(exclude_from_sim no)
+		(at 115.57 111.125 0)
+		(effects
+			(font
+				(size 3.9878 3.9878)
+				(thickness 0.7976)
+				(bold yes)
+			)
+			(justify left bottom)
+		)
+	)
 	(junction
 		(at 47.625 126.365)
@@
 		)
 	)
-	(rectangle
-		(start 219.71 67.945)
-		(end 282.575 113.03)
-		(stroke
-			(width 1)
-			(type default)
-		)
-		(fill
-			(type none)
-		)
-	)
-	(rectangle
-		(start 14.605 13.97)
-		(end 111.76 113.03)
-		(stroke
-			(width 1)
-			(type default)
-		)
-		(fill
-			(type none)
-		)
-	)
-	(rectangle
-		(start 14.605 166.37)
-		(end 67.31 195.58)
-		(stroke
-			(width 1)
-			(type default)
-		)
-		(fill
-			(type none)
-		)
-	)
-	(rectangle
-		(start 114.3 13.97)
-		(end 217.17 113.03)
-		(stroke
-			(width 1)
-			(type default)
-		)
-		(fill
-			(type none)
-		)
-	)
-	(rectangle
-		(start 14.605 116.205)
-		(end 282.575 163.195)
-		(stroke
-			(width 1)
-			(type default)
-		)
-		(fill
-			(type none)
-		)
-	)
-	(rectangle
-		(start 219.71 13.97)
-		(end 282.575 65.405)
-		(stroke
-			(width 1)
-			(type default)
-		)
-		(fill
-			(type none)
-		)
-	)
-	(rectangle
-		(start 70.485 166.37)
-		(end 123.19 195.58)
-		(stroke
-			(width 1)
-			(type default)
-		)
-		(fill
-			(type none)
-		)
-	)
-	(text "ESP32"
-		(exclude_from_sim no)
-		(at 15.875 111.125 0)
-		(effects
-			(font
-				(size 3.9878 3.9878)
-				(thickness 0.7976)
-				(bold yes)
-			)
-			(justify left bottom)
-		)
-	)
-	(text "RTC"
-		(exclude_from_sim no)
-		(at 220.98 63.5 0)
-		(effects
-			(font
-				(size 3.9878 3.9878)
-				(thickness 0.7976)
-				(bold yes)
-			)
-			(justify left bottom)
-		)
-	)
-	(text "POWER SUPPLY"
-		(exclude_from_sim no)
-		(at 15.875 161.925 0)
-		(effects
-			(font
-				(size 3.9878 3.9878)
-				(thickness 0.7976)
-				(bold yes)
-			)
-			(justify left bottom)
-		)
-	)
-	(text "DHT11"
-		(exclude_from_sim no)
-		(at 15.875 194.31 0)
-		(effects
-			(font
-				(size 3.9878 3.9878)
-				(thickness 0.7976)
-				(bold yes)
-			)
-			(justify left bottom)
-		)
-	)
-	(text "ILI9341"
-		(exclude_from_sim no)
-		(at 221.615 111.125 0)
-		(effects
-			(font
-				(size 3.9878 3.9878)
-				(thickness 0.7976)
-				(bold yes)
-			)
-			(justify left bottom)
-		)
-	)
-	(text "BUZZER"
-		(exclude_from_sim no)
-		(at 71.755 193.675 0)
-		(effects
-			(font
-				(size 3.9878 3.9878)
-				(thickness 0.7976)
-				(bold yes)
-			)
-			(justify left bottom)
-		)
-	)
-	(text "CP2102"
-		(exclude_from_sim no)
-		(at 115.57 111.125 0)
-		(effects
-			(font
-				(size 3.9878 3.9878)
-				(thickness 0.7976)
-				(bold yes)
-			)
-			(justify left bottom)
-		)
-	)
 	(global_label "ESP32_SDA"
 		(shape input)
@@
 			)
 		)
-		(property "Footprint" "footprints:ESP32-WROVER"
+		(property "Footprint" "Footprint-Kicad:ESP32-WROVER"
 			(at 65.405 70.485 0)
 			(effects
@@
 			)
 		)
-		(property "Footprint" "footprints:SNR4-2.54-15.5X12.0X5.5MM"
+		(property "Footprint" "Footprint-Kicad:SNR4-2.54-15.5X12.0X5.5MM"
 			(at 43.18 191.135 0)
 			(effects
@@
 			)
 		)
-		(property "Footprint" "footprints:BAT_CR1220_Holder"
+		(property "Footprint" "Footprint-Kicad:BAT_CR1220_Holder"
 			(at 267.97 25.781 90)
 			(effects
@@
 			)
 		)
-		(property "Footprint" "footprints:JST_EH_S2B-EH_1x02_P2.5mm_Horizontal"
+		(property "Footprint" "Footprint-Kicad:Connector_ZH_1x02_P1.25mm_Horizontal"
 			(at 80.645 97.155 0)
 			(effects
@@
 			)
 		)
-		(property "Footprint" "footprints:JST_EH_S2B-EH_1x02_P2.5mm_Horizontal"
+		(property "Footprint" "Footprint-Kicad:Connector_ZH_1x02_P1.25mm_Horizontal"
 			(at 66.04 128.905 90)
 			(effects
@@
 			)
 		)
-		(property "Footprint" "footprints:JST_EH_S3B-EH_1x03_P2.5mm_Horizontal"
+		(property "Footprint" "Footprint-Kicad:Connector_ZH_1x03_P1.25mm_Horizontal"
 			(at 246.38 92.71 0)
 			(effects
@@
 			)
 		)
-		(property "Footprint" "footprints:JST_EH_S2B-EH_1x02_P2.5mm_Horizontal"
+		(property "Footprint" "Footprint-Kicad:Connector_ZH_1x02_P1.25mm_Horizontal"
 			(at 47.625 128.905 90)
 			(effects
@@
 		)
 	)
+	(embedded_fonts no)
 )
